Commit message: robotic_gripper added

File: urdf/fanuc_crx10.urdf.xacro (robot description, xacro)
@@ -5,5 +5,4 @@
   <xacro:include filename="$(find fanuc_robot)/urdf/gazebo.xacro" />
   <xacro:include filename="$(find fanuc_robot)/urdf/robotic_gripper.xacro"/>
-  <!-- Inertial macro for simplified calculations -->
   <xacro:macro name="default_inertial" params="mass">
     <inertial>
@@ -12,5 +11,4 @@
     </inertial>
   </xacro:macro>
-  <!-- World link for Gazebo -->
   <link name="world"/>
   <link name="base_link">
@@ -212,5 +210,5 @@
   </joint>
   <xacro:robotic_gripper parent="tool0"/>
-  <!-- ros2_control configuration -->
+  <!-- ros2_control-->
   <ros2_control name="GazeboSystem" type="system">
     <hardware>
@@ -276,5 +274,5 @@
     </joint>
   </ros2_control>
-  <!-- Gazebo ros2_control plugin -->
+  <!-- gazebo ros2_control plugin -->
   <gazebo>
     <plugin filename="gz_ros2_control-system" name="gz_ros2_control::GazeboSimROS2ControlPlugin">

File: urdf/robotic_gripper.xacro (robot description, xacro)
@@ -2,5 +2,4 @@
 <robot xmlns:xacro="http://www.ros.org/wiki/xacro">
   <xacro:macro name="robotic_gripper" params="parent">
-    <!-- Base of gripper -->
     <link name="gripper_base_link">
       <visual>
@@ -23,5 +22,4 @@
       </inertial>
     </link>
-    <!-- Left finger -->
     <link name="left_finger">
       <visual>
@@ -44,6 +42,5 @@
       </inertial>
     </link>
-    <!-- Right finger -->
-   <link name="right_finger">
+    <link name="right_finger">
       <visual>
         <geometry>
@@ -65,25 +62,25 @@
       </inertial>
     </link>
-    <!-- Attach to robot tool0 -->
-  <joint name="gripper_mount" type="fixed">
-    <parent link="${parent}"/>
-    <child link="gripper_base_link"/>
-    <origin xyz="0 0 0.05" rpy="3.141592653589793 -1.5707963267948966 0"/>
-  </joint>
-    <!-- Left finger joint -->
+    <!-- Mount gripper to robot -->
+    <joint name="gripper_mount" type="fixed">
+      <parent link="${parent}"/>
+      <child link="gripper_base_link"/>
+      <origin xyz="0 0 0.05" rpy="0 0 0"/>
+    </joint>
+    <!-- Left finger prismatic -->
     <joint name="left_finger_joint" type="prismatic">
-        <parent link="gripper_base_link"/>
-        <child link="left_finger"/>
-        <origin xyz="0 0.02 0.01" rpy="0 0 0"/>
-        <axis xyz="0 1 0"/>
-        <limit lower="0.0" upper="0.04" effort="10" velocity="0.1"/>
+      <parent link="gripper_base_link"/>
+      <child link="left_finger"/>
+      <origin xyz="0 0.02 0" rpy="0 0 0"/>
+      <axis xyz="0 1 0"/>
+      <limit lower="0.0" upper="0.04" effort="10" velocity="0.1"/>
     </joint>
+    <!-- Right finger prismatic -->
     <joint name="right_finger_joint" type="prismatic">
-        <parent link="gripper_base_link"/>
-        <child link="right_finger"/>
-        <origin xyz="0 -0.02 0.01" rpy="0 0 0"/>
-        <axis xyz="0 -1 0"/>
-        <limit lower="0.0" upper="0.04" effort="10" velocity="0.1"/>
-        <mimic joint="left_finger_joint" multiplier="1.0"/>
+      <parent link="gripper_base_link"/>
+      <child link="right_finger"/>
+      <origin xyz="0 -0.02 0" rpy="0 0 0"/>
+      <axis xyz="0 -1 0"/>
+      <limit lower="0.0" upper="0.04" effort="10" velocity="0.1"/>
     </joint>
   </xacro:macro>
